Commit message: added the slam toolbox and created a test world

File: description/robot.urdf.xacro (robot description, xacro)
@@ -3,3 +3,4 @@
     <xacro:include filename= "robot_core.xacro"/>
     <xacro:include filename= "gazebo_control.xacro"/>
+    <xacro:include filename= "lidar.xacro"/>
 </robot>

File: description/robot_core.xacro (robot description, xacro)
@@ -14,6 +14,17 @@
     <color rgba="0 0 0 1"/>
     </material>
+    <material name="red">
+    <color rgba="1 0 0 1"/>
+    </material>
     <!--base link-->
     <link name="base_link">
+    </link>
+    <!-- BASE_FOOTPRINT LINK-->
+    <joint name = "base_footprint_joint" type="fixed">
+        <parent link="base_link"/>
+        <child link="base_footprint"/>
+        <origin xyz="0 0 0" rpy = "0 0 0"/>
+    </joint>
+    <link name = "base_footprint">
     </link>
     <!-- chassis link -->
